File: circuitry/single.kicad_sch (KiCad schematic)
At the start: 34 parts, among them J1 Conn_01x02, J2 Conn_01x03, P1 Touch_Pad, SW1 SW_Push, U1 MIC5225-5.0YM5, U2 ATtiny402-SS, U3 74LVC2GU04, Y1 16MHz

Commit message: Completed schematic and layout.
Parts:
- P1: now left out of the parts list
Changed lines of the file:
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@@
 	(title_block
 		(title "Capacitive Touch Test")
-		(date "2024-06-18")
+		(date "2024-07-27")
 		(rev "0")
 		(company "Ashlyn Black")
@@
 		(unit 1)
 		(exclude_from_sim no)
-		(in_bom yes)
+		(in_bom no)
 		(on_board yes)
 		(dnp no)
